File: Electron/V1/PCB/Thermocouple.brd (EAGLE design)
At the start: 95.8 x 33.6 mm, 30 parts, among them U1 MAX31855K, U2 ELECTRONDUALNAMED, U3 24LC512

Commit message: Tidied up identifiers and added BOM
Parts:
- R1: value (none) -> 1k5
- R3, R4: value 2k -> 4k7
- R5: value (none) -> 10k
- renumbered U$2 to JP2
Changed lines of the file:
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@@
 <grid distance="0.025" unitdist="inch" unit="inch" style="lines" multiple="1" display="yes" altdistance="0.0125" altunitdist="inch" altunit="inch"/>
 <layers>
-<layer number="1" name="Top" color="4" fill="1" visible="no" active="yes"/>
+<layer number="1" name="Top" color="4" fill="1" visible="yes" active="yes"/>
 <layer number="2" name="Route2" color="1" fill="3" visible="no" active="no"/>
 <layer number="3" name="Route3" color="4" fill="3" visible="no" active="no"/>
@@
 <layer number="23" name="tOrigins" color="15" fill="1" visible="yes" active="yes"/>
 <layer number="24" name="bOrigins" color="15" fill="1" visible="yes" active="yes"/>
-<layer number="25" name="tNames" color="7" fill="1" visible="no" active="yes"/>
+<layer number="25" name="tNames" color="7" fill="1" visible="yes" active="yes"/>
 <layer number="26" name="bNames" color="7" fill="1" visible="yes" active="yes"/>
-<layer number="27" name="tValues" color="7" fill="1" visible="no" active="yes"/>
+<layer number="27" name="tValues" color="7" fill="1" visible="yes" active="yes"/>
 <layer number="28" name="bValues" color="7" fill="1" visible="yes" active="yes"/>
 <layer number="29" name="tStop" color="7" fill="3" visible="yes" active="yes"/>
@@
 <attribute name="VALUE" x="92.71" y="29.21" size="1.27" layer="28" rot="MR180"/>
 </element>
-<element name="R1" library="SparkFun-Resistors" package="1206" value="" x="83.185" y="27.305" locked="yes" smashed="yes" rot="MR0">
+<element name="R1" library="SparkFun-Resistors" package="1206" value="1k5" x="83.185" y="27.305" locked="yes" smashed="yes" rot="MR0">
 <attribute name="NAME" x="85.725" y="24.638" size="1.27" layer="26" rot="MR0"/>
 <attribute name="VALUE" x="84.582" y="25.781" size="0.4064" layer="28" rot="MR0"/>
@@
 <attribute name="NAME" x="39.243" y="10.3505" size="1.27" layer="25"/>
 </element>
-<element name="R3" library="SparkFun-Resistors" package="0805" value="2k" x="47.625" y="17.145" locked="yes" smashed="yes" rot="R180">
+<element name="R3" library="SparkFun-Resistors" package="0805" value="4k7" x="47.625" y="17.145" locked="yes" smashed="yes" rot="R180">
 <attribute name="NAME" x="45.847" y="17.5895" size="1.27" layer="25" rot="R180"/>
 </element>
-<element name="R4" library="SparkFun-Resistors" package="0805" value="2k" x="45.085" y="19.05" locked="yes" smashed="yes" rot="R180">
+<element name="R4" library="SparkFun-Resistors" package="0805" value="4k7" x="45.085" y="19.05" locked="yes" smashed="yes" rot="R180">
 <attribute name="NAME" x="43.307" y="19.4945" size="1.27" layer="25" rot="R180"/>
 </element>
-<element name="U$2" library="Tinamous" package="THERMOCOUPLE_SOCKET_K-TYPE" value="THERMOCOUPLE_SOCKET_K-TYPE" x="90.805" y="4.445" locked="yes" smashed="yes"/>
-<element name="R5" library="SparkFun-Resistors" package="0805" value="" x="75.565" y="16.51" locked="yes" smashed="yes">
+<element name="JP2" library="Tinamous" package="THERMOCOUPLE_SOCKET_K-TYPE" value="THERMOCOUPLE_SOCKET_K-TYPE" x="90.805" y="4.445" locked="yes" smashed="yes"/>
+<element name="R5" library="SparkFun-Resistors" package="0805" value="10k" x="75.565" y="16.51" locked="yes" smashed="yes">
 <attribute name="NAME" x="77.343" y="16.0655" size="1.27" layer="25"/>
 <attribute name="VALUE" x="74.549" y="15.113" size="0.4064" layer="27"/>
@@
 <contactref element="L6" pad="1"/>
 <contactref element="JP1" pad="P1"/>
-<contactref element="U$2" pad="P$-"/>
+<contactref element="JP2" pad="P$-"/>
 <wire x1="85.99" y1="11.43" x2="94.805" y2="11.43" width="1.016" layer="1"/>
 <wire x1="94.805" y1="11.43" x2="94.805" y2="8.945" width="1.016" layer="1"/>
@@
 <contactref element="JP1" pad="P2"/>
 <contactref element="L5" pad="1"/>
-<contactref element="U$2" pad="P$+"/>
+<contactref element="JP2" pad="P$+"/>
 <wire x1="85.99" y1="13.97" x2="94.805" y2="13.97" width="1.016" layer="1"/>
 <wire x1="94.805" y1="13.97" x2="94.805" y2="16.945" width="1.016" layer="1"/>
